Commit message: update

File: dm_robotarm_description/urdf/dm_arm.urdf (robot description, URDF)
Before this commit: robot dm_arm, 10 links, 9 joints
Links:
- link base_link: geometry collision mesh filename=file://$(find dm_robotarm_description)/meshes/base_link.STL; visual mesh filename=file://$(find dm_robotarm_description)/meshes/base_link.STL
- link dm_hand: geometry collision mesh filename=file://$(find dm_robotarm_description)/meshes/dm_hand.STL; visual mesh filename=file://$(find dm_robotarm_description)/meshes/dm_hand.STL
- link dm_left_hand: geometry collision mesh filename=file://$(find dm_robotarm_description)/meshes/dm_left_hand.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; visual mesh filename=file://$(find dm_robotarm_description)/meshes/dm_left_hand.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
- link dm_right_hand: geometry collision mesh filename=file://$(find dm_robotarm_description)/meshes/dm_right_hand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; visual mesh filename=file://$(find dm_robotarm_description)/meshes/dm_right_hand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
- link link1: geometry collision mesh filename=file://$(find dm_robotarm_description)/meshes/link1.STL; visual mesh filename=file://$(find dm_robotarm_description)/meshes/link1.STL
- link link2: geometry collision mesh filename=file://$(find dm_robotarm_description)/meshes/link2.STL; visual mesh filename=file://$(find dm_robotarm_description)/meshes/link2.STL
- link link3: geometry collision mesh filename=file://$(find dm_robotarm_description)/meshes/link3.STL; visual mesh filename=file://$(find dm_robotarm_description)/meshes/link3.STL
- link link4: geometry collision mesh filename=file://$(find dm_robotarm_description)/meshes/link4.STL; visual mesh filename=file://$(find dm_robotarm_description)/meshes/link4.STL
- link link5: geometry collision mesh filename=file://$(find dm_robotarm_description)/meshes/link5.STL; visual mesh filename=file://$(find dm_robotarm_description)/meshes/link5.STL
- link link6: geometry collision mesh filename=file://$(find dm_robotarm_description)/meshes/link6.STL; visual mesh filename=file://$(find dm_robotarm_description)/meshes/link6.STL

Commit message: add mujoco

File: dm_robotarm_description/urdf/dm_arm.urdf (robot description, URDF)
Before this commit: robot dm_arm, 10 links, 9 joints
Links:
- link base_link: geometry collision mesh filename=package://dm_robotarm_description/meshes/base_link.STL; visual mesh filename=package://dm_robotarm_description/meshes/base_link.STL
- link dm_hand: geometry collision mesh filename=package://dm_robotarm_description/meshes/dm_hand.STL; visual mesh filename=package://dm_robotarm_description/meshes/dm_hand.STL
- link dm_left_hand: geometry collision mesh filename=package://dm_robotarm_description/meshes/dm_left_hand.STL; visual mesh filename=package://dm_robotarm_description/meshes/dm_left_hand.STL
- link dm_right_hand: geometry collision mesh filename=package://dm_robotarm_description/meshes/dm_right_hand.STL; visual mesh filename=package://dm_robotarm_description/meshes/dm_right_hand.STL
- link link1: geometry collision mesh filename=package://dm_robotarm_description/meshes/link1.STL; visual mesh filename=package://dm_robotarm_description/meshes/link1.STL
- link link2: geometry collision mesh filename=package://dm_robotarm_description/meshes/link2.STL; visual mesh filename=package://dm_robotarm_description/meshes/link2.STL
- link link3: geometry collision mesh filename=package://dm_robotarm_description/meshes/link3.STL; visual mesh filename=package://dm_robotarm_description/meshes/link3.STL
- link link4: geometry collision mesh filename=package://dm_robotarm_description/meshes/link4.STL; visual mesh filename=package://dm_robotarm_description/meshes/link4.STL
- link link5: geometry collision mesh filename=package://dm_robotarm_description/meshes/link5.STL; visual mesh filename=package://dm_robotarm_description/meshes/link5.STL
- link link6: geometry collision mesh filename=package://dm_robotarm_description/meshes/link6.STL; visual mesh filename=package://dm_robotarm_description/meshes/link6.STL
